File: v1.brd (EAGLE design)
At the start: 33 x 16 mm, 17 parts, among them IC1 FT232RL, Q1 IRLML6402, U1 HM-MOD-UART-AW-SH-2, X1 A-USB A-LP-SMT-C

Commit message: Fix not connected pin TEST
Connections:
- net GND: now also IC1.26
Changed lines of the file:
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@@
 <via x="17" y="10" extent="1-16" drill="0.35"/>
 <via x="20.4" y="7.9" extent="1-16" drill="0.35"/>
+<contactref element="IC1" pad="26"/>
 </signal>
 <signal name="VUSB">
