File: v1.sch (EAGLE design)
At the start: 17 parts, among them IC1 FT232RL, Q1 IRLML6402, U1 HM-MOD-UART-AW-SH-2, X1 A-USB A-LP-SMT-C

Commit message: Fix not connected pin TEST
Connections:
- net GND: now also IC1.TEST
Changed lines of the file:
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@@
 <wire x1="167.64" y1="63.5" x2="170.18" y2="63.5" width="0.1524" layer="91"/>
 <junction x="170.18" y="63.5"/>
+<pinref part="IC1" gate="1" pin="TEST"/>
+<wire x1="167.64" y1="73.66" x2="170.18" y2="73.66" width="0.1524" layer="91"/>
+<wire x1="170.18" y1="73.66" x2="170.18" y2="68.58" width="0.1524" layer="91"/>
+<junction x="170.18" y="68.58"/>
 </segment>
 <segment>
